File: Fennec6800.kicad_sch (KiCad schematic)
At the start: 115 parts, among them J1 Barrel_Jack, J2 DB25_Male, J3 Expansion Connector, J4 DB25_Male, Q1 2N3904-AP, SW1 SW_DIP_x06, SW2 SW_DIP_x06, SW3 SW_Push, SW4 SW_DPDT_x2, U1 74LS00, U10 74LS245, U11 MC6800, U12 74LS244, U13 74LS244, U14 74LS244, U15 74LS138, U16 74LS138, U17 P2114, U18 P2114, U19 P2114, U2 74LS04, U20 P2114, U21 2716, U22 P2114, U23 P2114, U24 P2114, U25 P2114, U26 P2114, U27 P2114, U28 P2114, U29 P2114, U3 74LS193, U30 P2114, U31 P2114, U32 P2114, U33 P2114, U34 MAX232, U35 MAX232, U36 74LS30, U37 NE555P, U4 74LS73, U5 74LS02, U6 74LS74, U7 MC6850, U8 MC6850, U9 74LS245, X1 ACO-1.8432MHz

Commit message: Rename Project from 77Project. Add documentation
Parts:
- added C55, C56: 1uF, Capacitor_THT:C_Disc_D3.8mm_W2.6mm_P2.50mm, symbol Device:C_Small
- added D2: 1N4148, symbol Device:D
- added R13: 10k, Resistor_THT:R_Axial_DIN0207_L6.3mm_D2.5mm_P10.16mm_Horizontal, symbol Device:R_US
Connections:
- net CLK: no longer SW1.7, SW2.7
- net CPUA15: now also U9.19 (CE)
- net E_Phi2: no longer U10.19 (CE), U9.19 (CE)
- net GND: now also C55.2, C56.2; no longer R8.1
- net VCC: now also R8.1, C55.1, C56.1, R13.2
- net ~{EXP0}: now also D2.1 (K)
- net FULLCLK: now reaches U6.3 (C), X1.8 (OUT)
- net FULLCLK: now also SW1.7, SW2.7
- net ~{BEN}: now reaches J3.32 (Pin_32)
- net ~{BEN}: now also U10.19 (CE), D2.2 (A), R13.1
- no-connect marks 50 -> 49
Other:
- note added: "*"
- note added: "Bodge for data bus buffer"
- note added: "Expansion cards must assert ~{BEN} to access the data bus (Open collector input)"
- note added: "Schotkey diodes may be a good idea but silicon ones should be low enough for the LS245 input low voltage (0.8v max)"

Commit message: Updated manual and schematic
Other:
- company: (none) -> Chartreuse
- title: (none) -> Fennec 6800
